File: electricpanelinput.sch (KiCad schematic (older format))
At the start: 25 parts, among them J1 5V, J10 Blu-, J11 Blu+, J12 Vic-, J13 Vic+, J2 12V, J3 VDC, J4 GND, J5 CRE, J6 BlueSun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

Commit message: 1 Layer PCB, input resistor protection
Parts:
- added R1, R2, R3: 1k, Resistor_THT:R_Axial_DIN0207_L6.3mm_D2.5mm_P10.16mm_Horizontal, symbol Device:R
- J10, J11, J12, J13, J8, J9: footprint Connector_PinHeader_2.54mm:PinHeader_1x01_P2.54mm_Vertical -> Connector_PinHeader_2.54mm:PinHeader_1x02_P2.54mm_Vertical; symbol Connector_Generic:Conn_01x01 -> Connector_Generic:Conn_01x02
- JUSB1: symbol Connector:USB_A -> electricpanelinput-rescue:USB_A-Connector
Connections:
- net 0: now also J10.2 (Pin_2), J12.2 (Pin_2), J9.2 (Pin_2)
- net Blu+: now also J11.2 (Pin_2)
- net CRE+: now also J8.2 (Pin_2)
- net OBlu: now also R2.2; no longer Relay2.1
- net OCRE: now also R1.2; no longer Relay1.1
- net OVic: now also R3.2; no longer Relay3.1
- net Vic+: now also J13.2 (Pin_2)
- new net: R1.1, Relay1.1
- new net: R2.1, Relay2.1
- new net: R3.1, Relay3.1
Changed lines of the file:
@@
 $EndComp
 $Comp
-L Connector:USB_A JUSB1
+L electricpanelinput-rescue:USB_A-Connector JUSB1
 U 1 1 5F3256A2
 P 2150 1500
@@
 $EndComp
 Wire Wire Line
-	6600 5250 6600 5800
-Wire Wire Line
 	6600 5800 5900 5800
 Wire Wire Line
@@
 Connection ~ 5900 6250
 Wire Wire Line
-	9300 5250 9300 5700
-Wire Wire Line
 	9300 5700 8600 5700
 Wire Wire Line
@@
 	3400 6200 3400 6300
 Connection ~ 3400 6200
-Wire Wire Line
-	4200 5700 3400 5700
-$Comp
-L Relay:SANYOU_SRD_Form_C Relay1
-U 1 1 5F32050B
-P 4000 4950
-F 0 "Relay1" H 4430 4996 50  0000 L CNN
-F 1 "SANYOU_SRD_Form_C" H 4430 4905 50  0000 L CNN
-F 2 "Relay_THT:Relay_SPDT_SANYOU_SRD_Series_Form_C" H 4450 4900 50  0001 L CNN
-F 3 "http://www.sanyourelay.ca/public/products/pdf/SRD.pdf" H 4000 4950 50  0001 C CNN
-	1    4000 4950
-	1    0    0    -1
-$EndComp
 $Comp
 L pspice:0 #GND0101
@@
 	3800 5250 3800 5450
 Wire Wire Line
-	4200 5250 4200 5700
-Wire Wire Line
 	2450 5250 2450 4350
 Wire Wire Line
@@
 Connection ~ 4100 4350
 Wire Wire Line
-	4100 4350 5800 4350
+	4100 4350 5700 4350
 Wire Wire Line
 	6500 4650 6500 4350
 Connection ~ 6500 4350
 Wire Wire Line
-	6500 4350 8500 4350
+	6500 4350 8400 4350
 Wire Wire Line
 	9200 4650 9200 4350
@@
 1.0\n
 Wire Wire Line
-	3000 4350 3500 4350
+	3000 4350 3400 4350
 Connection ~ 3000 4350
 Wire Wire Line
@@
 	3900 1500 3900 1600
 $Comp
-L Connector_Generic:Conn_01x01 J10
+L Connector_Generic:Conn_01x02 J10
 U 1 1 5F333494
 P 5800 4650
 F 0 "J10" V 5672 4730 50  0000 L CNN
 F 1 "Blu-" V 5763 4730 50  0000 L CNN
-F 2 "Connector_PinHeader_2.54mm:PinHeader_1x01_P2.54mm_Vertical" H 5800 4650 50  0001 C CNN
+F 2 "Connector_PinHeader_2.54mm:PinHeader_1x02_P2.54mm_Vertical" H 5800 4650 50  0001 C CNN
 F 3 "~" H 5800 4650 50  0001 C CNN
 	1    5800 4650
@@
 $EndComp
 $Comp
-L Connector_Generic:Conn_01x01 J11
+L Connector_Generic:Conn_01x02 J11
 U 1 1 5F334231
 P 5800 5050
 F 0 "J11" V 5764 4962 50  0000 R CNN
 F 1 "Blu+" V 5673 4962 50  0000 R CNN
-F 2 "Connector_PinHeader_2.54mm:PinHeader_1x01_P2.54mm_Vertical" H 5800 5050 50  0001 C CNN
+F 2 "Connector_PinHeader_2.54mm:PinHeader_1x02_P2.54mm_Vertical" H 5800 5050 50  0001 C CNN
 F 3 "~" H 5800 5050 50  0001 C CNN
 	1    5800 5050
@@
 $EndComp
 $Comp
-L Connector_Generic:Conn_01x01 J9
+L Connector_Generic:Conn_01x02 J9
 U 1 1 5F33543C
-P 3500 4550
-F 0 "J9" V 3372 4630 50  0000 L CNN
-F 1 "CRE-" V 3463 4630 50  0000 L CNN
-F 2 "Connector_PinHeader_2.54mm:PinHeader_1x01_P2.54mm_Vertical" H 3500 4550 50  0001 C CNN
-F 3 "~" H 3500 4550 50  0001 C CNN
-	1    3500 4550
+P 3500 4600
+F 0 "J9" V 3372 4680 50  0000 L CNN
+F 1 "CRE-" V 3463 4680 50  0000 L CNN
+F 2 "Connector_PinHeader_2.54mm:PinHeader_1x02_P2.54mm_Vertical" H 3500 4600 50  0001 C CNN
+F 3 "~" H 3500 4600 50  0001 C CNN
+	1    3500 4600
 	0    1    1    0
 $EndComp
 $Comp
-L Connector_Generic:Conn_01x01 J8
+L Connector_Generic:Conn_01x02 J8
 U 1 1 5F33650C
-P 3450 5000
-F 0 "J8" V 3414 4912 50  0000 R CNN
-F 1 "CRE+" V 3323 4912 50  0000 R CNN
-F 2 "Connector_PinHeader_2.54mm:PinHeader_1x01_P2.54mm_Vertical" H 3450 5000 50  0001 C CNN
-F 3 "~" H 3450 5000 50  0001 C CNN
-	1    3450 5000
+P 3400 5000
+F 0 "J8" V 3364 4912 50  0000 R CNN
+F 1 "CRE+" V 3273 4912 50  0000 R CNN
+F 2 "Connector_PinHeader_2.54mm:PinHeader_1x02_P2.54mm_Vertical" H 3400 5000 50  0001 C CNN
+F 3 "~" H 3400 5000 50  0001 C CNN
+	1    3400 5000
 	0    -1   -1   0
 $EndComp
 $Comp
-L Connector_Generic:Conn_01x01 J12
+L Connector_Generic:Conn_01x02 J12
 U 1 1 5F33818C
 P 8500 4600
 F 0 "J12" V 8372 4680 50  0000 L CNN
 F 1 "Vic-" V 8463 4680 50  0000 L CNN
-F 2 "Connector_PinHeader_2.54mm:PinHeader_1x01_P2.54mm_Vertical" H 8500 4600 50  0001 C CNN
+F 2 "Connector_PinHeader_2.54mm:PinHeader_1x02_P2.54mm_Vertical" H 8500 4600 50  0001 C CNN
 F 3 "~" H 8500 4600 50  0001 C CNN
 	1    8500 4600
@@
 $EndComp
 $Comp
-L Connector_Generic:Conn_01x01 J13
+L Connector_Generic:Conn_01x02 J13
 U 1 1 5F338CD6
 P 8500 4950
 F 0 "J13" V 8464 4862 50  0000 R CNN
 F 1 "Vic+" V 8373 4862 50  0000 R CNN
-F 2 "Connector_PinHeader_2.54mm:PinHeader_1x01_P2.54mm_Vertical" H 8500 4950 50  0001 C CNN
+F 2 "Connector_PinHeader_2.54mm:PinHeader_1x02_P2.54mm_Vertical" H 8500 4950 50  0001 C CNN
 F 3 "~" H 8500 4950 50  0001 C CNN
 	1    8500 4950
 	0    -1   -1   0
 $EndComp
-Connection ~ 3500 4350
 Wire Wire Line
 	3500 4350 3800 4350
 Wire Wire Line
 	3300 3300 3300 5550
-Wire Wire Line
-	3450 5200 3650 5200
 Wire Wire Line
 	3650 5200 3650 5450
@@
 	5800 5250 5800 5350
 Wire Wire Line
-	5800 5350 6200 5350
+	5800 5350 5900 5350
 Connection ~ 6200 5350
 Wire Wire Line
@@
 	8500 5150 8500 5250
 Wire Wire Line
-	8500 5250 8900 5250
+	8500 5250 8600 5250
 Connection ~ 8900 5250
 Wire Wire Line
@@
 	6900 3500 6900 3600
 Connection ~ 6900 3600
+$Comp
+L Device:R R1
+U 1 1 5F90B25D
+P 4200 5500
+F 0 "R1" H 4270 5546 50  0000 L CNN
+F 1 "1k" H 4270 5455 50  0000 L CNN
+F 2 "Resistor_THT:R_Axial_DIN0207_L6.3mm_D2.5mm_P10.16mm_Horizontal" V 4130 5500 50  0001 C CNN
+F 3 "~" H 4200 5500 50  0001 C CNN
+	1    4200 5500
+	1    0    0    -1
+$EndComp
+$Comp
+L Device:R R2
+U 1 1 5F90BC54
+P 6600 5550
+F 0 "R2" H 6670 5596 50  0000 L CNN
+F 1 "1k" H 6670 5505 50  0000 L CNN
+F 2 "Resistor_THT:R_Axial_DIN0207_L6.3mm_D2.5mm_P10.16mm_Horizontal" V 6530 5550 50  0001 C CNN
+F 3 "~" H 6600 5550 50  0001 C CNN
+	1    6600 5550
+	1    0    0    -1
+$EndComp
+$Comp
+L Relay:SANYOU_SRD_Form_C Relay1
+U 1 1 5F32050B
+P 4000 4950
+F 0 "Relay1" H 4430 4996 50  0000 L CNN
+F 1 "SANYOU_SRD_Form_C" H 4430 4905 50  0000 L CNN
+F 2 "Relay_THT:Relay_SPDT_SANYOU_SRD_Series_Form_C" H 4450 4900 50  0001 L CNN
+F 3 "http://www.sanyourelay.ca/public/products/pdf/SRD.pdf" H 4000 4950 50  0001 C CNN
+	1    4000 4950
+	1    0    0    -1
+$EndComp
+Wire Wire Line
+	4200 5700 3400 5700
+Wire Wire Line
+	9300 5650 9300 5700
+Wire Wire Line
+	9300 5250 9300 5350
+Wire Wire Line
+	6600 5250 6600 5400
+Wire Wire Line
+	6600 5700 6600 5800
+Wire Wire Line
+	4200 5250 4200 5350
+Wire Wire Line
+	4200 5650 4200 5700
+$Comp
+L Device:R R3
+U 1 1 5F90C5CB
+P 9300 5500
+F 0 "R3" H 9370 5546 50  0000 L CNN
+F 1 "1k" H 9370 5455 50  0000 L CNN
+F 2 "Resistor_THT:R_Axial_DIN0207_L6.3mm_D2.5mm_P10.16mm_Horizontal" V 9230 5500 50  0001 C CNN
+F 3 "~" H 9300 5500 50  0001 C CNN
+	1    9300 5500
+	1    0    0    -1
+$EndComp
+Wire Wire Line
+	8600 5150 8600 5250
+Connection ~ 8600 5250
+Wire Wire Line
+	8600 5250 8900 5250
+Wire Wire Line
+	8400 4400 8400 4350
+Connection ~ 8400 4350
+Wire Wire Line
+	8400 4350 8500 4350
+Wire Wire Line
+	5900 5250 5900 5350
+Connection ~ 5900 5350
+Wire Wire Line
+	5900 5350 6200 5350
+Wire Wire Line
+	5700 4450 5700 4350
+Connection ~ 5700 4350
+Wire Wire Line
+	5700 4350 5800 4350
+Wire Wire Line
+	3400 4400 3400 4350
+Wire Wire Line
+	3500 4350 3500 4400
+Wire Wire Line
+	3500 4350 3400 4350
+Connection ~ 3500 4350
+Connection ~ 3400 4350
+Connection ~ 3500 5200
+Wire Wire Line
+	3500 5200 3650 5200
+Wire Wire Line
+	3400 5200 3500 5200
 $EndSCHEMATC
